File: esp32/nixie-display/anode_drivers.sch (KiCad schematic (older format))
At the start: 43 parts, among them J2 Conn_01x10_Male, Q1 Q_NPN_CBE, Q10 Q_PNP_CBE, Q11 Q_NPN_CBE, Q12 Q_PNP_CBE, Q13 Q_NPN_CBE, Q14 Q_PNP_CBE, Q2 Q_PNP_CBE, Q3 Q_NPN_CBE, Q4 Q_PNP_CBE, Q5 Q_NPN_CBE, Q6 Q_PNP_CBE, Q7 Q_NPN_CBE, Q8 Q_PNP_CBE, Q9 Q_NPN_CBE

Commit message: Improved grounding New Anode Drivers
[git-p4: depot-paths = "//depot/nixiestat/": change = 328]
Parts:
- removed J2: Conn_01x10_Male, Connector_PinHeader_2.54mm:PinHeader_1x10_P2.54mm_Vertical, symbol Connector:Conn_01x10_Male
- added J2: Conn_02x10_Odd_Even, Connector_PinHeader_2.54mm:PinHeader_2x10_P2.54mm_Vertical, symbol Connector_Generic:Conn_02x10_Odd_Even
- added R1, R13, R17, R25, R5, R9: 3.3K, Resistor_SMD:R_0805_2012Metric_Pad1.20x1.40mm_HandSolder, symbol Device:R_US
- Q1, Q11, Q13, Q3, Q5, Q7, Q9: value Q_NPN_CBE -> MPSA42; symbol Device:Q_NPN_CBE -> Device:Q_NPN_EBC
- Q10, Q12, Q14, Q2, Q4, Q6, Q8: value Q_PNP_CBE -> MPSA92; symbol Device:Q_PNP_CBE -> Device:Q_PNP_EBC
- R12: renamed from R9; footprint Resistor_SMD:R_0805_2012Metric_Pad1.20x1.40mm_HandSolder -> Resistor_SMD:R_1206_3216Metric_Pad1.30x1.75mm_HandSolder
- R16: renamed from R12; footprint Resistor_SMD:R_0805_2012Metric_Pad1.20x1.40mm_HandSolder -> Resistor_SMD:R_1206_3216Metric_Pad1.30x1.75mm_HandSolder
- R20: renamed from R15; footprint Resistor_SMD:R_0805_2012Metric_Pad1.20x1.40mm_HandSolder -> Resistor_SMD:R_1206_3216Metric_Pad1.30x1.75mm_HandSolder
- R21: value 35K -> 3.3K
- R24: renamed from R18; footprint Resistor_SMD:R_0805_2012Metric_Pad1.20x1.40mm_HandSolder -> Resistor_SMD:R_1206_3216Metric_Pad1.30x1.75mm_HandSolder
- R4: renamed from R3; footprint Resistor_SMD:R_0805_2012Metric_Pad1.20x1.40mm_HandSolder -> Resistor_SMD:R_1206_3216Metric_Pad1.30x1.75mm_HandSolder
- R8: renamed from R6; footprint Resistor_SMD:R_0805_2012Metric_Pad1.20x1.40mm_HandSolder -> Resistor_SMD:R_1206_3216Metric_Pad1.30x1.75mm_HandSolder
- renumbered R7 to R10, R8 to R11, R10 to R14, R11 to R15, R13 to R18, R14 to R19, R1 to R2, R16 to R22, R17 to R23, R19 to R26, R20 to R27, R2 to R3, R4 to R6, R5 to R7
Connections:
- net 160V: now also Q10.1 (E), Q12.1 (E), Q14.1 (E), Q2.1 (E), Q4.1 (E), Q6.1 (E), Q8.1 (E); no longer Q10.3 (E), Q12.3 (E), Q14.3 (E), Q2.3 (E), Q4.3 (E), Q6.3 (E), Q8.3 (E)
- net GNDREF: now also J2.1 (Pin_1), J2.11 (Pin_11), J2.13 (Pin_13), J2.15 (Pin_15), J2.17 (Pin_17), J2.19 (Pin_19), J2.20 (Pin_20), J2.3 (Pin_3), J2.5 (Pin_5), J2.7 (Pin_7), J2.9 (Pin_9)
- net HV_DISABLE: now also J2.16 (Pin_16)
- net VCC: now also J2.18 (Pin_18)
- net dig6: now also Q14.3 (C); no longer R21.1
- net idig0: now also J2.2 (Pin_2), R1.2; no longer Q1.2 (B)
- net idig1: now also J2.4 (Pin_4), R5.2; no longer Q3.2 (B)
- net idig2: now also J2.6 (Pin_6), R9.2; no longer Q5.2 (B)
- net idig3: now also J2.8 (Pin_8), R13.2; no longer Q7.2 (B)
- net idig4: now also J2.10 (Pin_10), R17.2; no longer Q9.2 (B)
- net idig5: now also R21.2, J2.12 (Pin_12); no longer Q11.2 (B)
- net idig6: now also J2.14 (Pin_14), R25.2; no longer Q13.2 (B)
- net at R3.1: now also Q1.1 (E); no longer Q1.3 (E)
- net at R4.2: now also Q2.3 (C); no longer Q2.1 (C)
- net at Q2.2 (B), R2.2: now also Q1.3 (C); no longer Q1.1 (C)
- net at R7.1: now also Q3.1 (E); no longer Q3.3 (E)
- net at R8.2: now also Q4.3 (C); no longer Q4.1 (C)
- net at Q4.2 (B), R6.2: now also Q3.3 (C); no longer Q3.1 (C)
- net at R11.1: now also Q5.1 (E); no longer Q5.3 (E)
- net at R12.2: now also Q6.3 (C); no longer Q6.1 (C)
- net at Q6.2 (B), R10.2: now also Q5.3 (C); no longer Q5.1 (C)
- net at R15.1: now also Q7.1 (E); no longer Q7.3 (E)
- net at R16.2: now also Q8.3 (C); no longer Q8.1 (C)
- net at Q8.2 (B), R14.2: now also Q7.3 (C); no longer Q7.1 (C)
- net at R19.1: now also Q9.1 (E); no longer Q9.3 (E)
- net at R20.2: now also Q10.3 (C); no longer Q10.1 (C)
- net at Q10.2 (B), R18.2: now also Q9.3 (C); no longer Q9.1 (C)
- net at R23.1: now also Q11.1 (E); no longer Q11.3 (E)
- net at R24.2: now also Q12.3 (C); no longer Q12.1 (C)
- net at Q12.2 (B), R22.2: now also Q11.3 (C); no longer Q11.1 (C)
- net at R27.1: now also Q13.1 (E); no longer Q13.3 (E)
- net at Q14.2 (B), R26.2: now also Q13.3 (C); no longer Q13.1 (C)
- new net: Q1.2 (B), R1.1
- new net: Q7.2 (B), R13.1
- new net: Q13.2 (B), R25.1
- new net: Q9.2 (B), R17.1
- new net: Q3.2 (B), R5.1
- new net: Q5.2 (B), R9.1
- new net: Q11.2 (B), R21.1
Other:
- moved on the sheet: Q1, Q10, Q11, Q12, Q13, Q14, Q2, Q3, Q4, Q5, Q6, Q7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

Commit message: New Zen design
[git-p4: depot-paths = "//depot/nixiestat/": change = 356]
Parts:
- removed Q1, Q11: MPSA42, Package_TO_SOT_THT:TO-92L_Inline_Wide, symbol Device:Q_NPN_EBC
- removed Q12, Q2: MPSA92, Package_TO_SOT_THT:TO-92L_Inline_Wide, symbol Device:Q_PNP_EBC
- removed R1, R21, R23, R3: 3.3K, Resistor_SMD:R_0805_2012Metric_Pad1.20x1.40mm_HandSolder, symbol Device:R_US
- removed R2, R22: 100K, Resistor_SMD:R_0805_2012Metric_Pad1.20x1.40mm_HandSolder, symbol Device:R_US
- removed R24, R4: 22K, Resistor_SMD:R_1206_3216Metric_Pad1.30x1.75mm_HandSolder, symbol Device:R_US
- removed V2, V7: 160V, symbol croftj:160V
- renumbered Q3 to Q1, Q4 to Q2, Q5 to Q3, Q6 to Q4, Q7 to Q5, Q8 to Q6, Q13 to Q7, Q14 to Q8, R5 to R1, R14 to R10, R15 to R11, R16 to R12, R25 to R13, R26 to R14, R27 to R15, R17 to R16, R18 to R17, R19 to R18, R20 to R19, R6 to R2, R7 to R3, R8 to R4, R9 to R5, R10 to R6, R11 to R7, R12 to R8, R13 to R9
Connections:
- net dig6 is gone; now on net dig4: Q8.3 (C)
- net dig0: now also R4.1
- net dig1: now also R8.1; no longer R4.1
- net dig2: now also R12.1; no longer R8.1
- net dig3: now also R19.1; no longer R12.1
- net dig4: no longer R19.1
- net idig0: now also R1.2
- net idig1: now also R5.2; no longer R1.2
- net idig2: now also R9.2; no longer R5.2
- net idig3: now also R16.2; no longer R9.2
- net idig4: now also R13.2; no longer R16.2
- net idig5: no longer names the net of J2.12 (Pin_12)
- net idig6: no longer names the net of J2.14 (Pin_14)
- net idig6: no longer R13.2
Other:
- moved on the sheet: J2, Q1, Q10, Q2, Q3, Q4, Q5, Q6, Q7, Q8, Q9, R1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
