File: esp32/nixie-display/nixie-display.kicad_pcb (KiCad board)
At the start: 2 copper layers, 99.9 x 69.8 mm, 88 parts, among them J1 Conn_02x10_Odd_Even, J2 Conn_02x10_Odd_Even, Q1 MPSA42, Q10 MPSA92, Q11 MPSA42, Q12 MPSA92, Q13 MPSA42, Q14 MPSA92, Q15 IRLS640, Q2 MPSA92, Q3 MPSA42, Q4 MPSA92, Q5 MPSA42, Q6 MPSA92, Q7 MPSA42, Q8 MPSA92, Q9 MPSA42, U1 MAX1771, U2 L78L05_TO92

Commit message: Design Rule cleanup
[git-p4: depot-paths = "//depot/nixiestat/": change = 331]
Routing:
- net dig0: track 26.6 -> 25.6 mm
- net idig1: track 87.4 -> 86.8 mm

Commit message: Further ground work
[git-p4: depot-paths = "//depot/nixiestat/": change = 333]
Parts:
- moved R4 0.34 mm to (130.2, 75.1)
Routing:
- net GNDREF: track 459.7 -> 557.8 mm, vias 38 -> 112
- net dig6: track 194.3 -> 195.7 mm
- net dig0: track 25.6 -> 26.2 mm

Commit message: New Zen design
[git-p4: depot-paths = "//depot/nixiestat/": change = 356]
Parts:
- removed Nx5, Nx6: in17, croftj:in17
- removed Q11, Q13: MPSA42, Package_TO_SOT_THT:TO-92L_Inline_Wide
- removed Q12, Q14: MPSA92, Package_TO_SOT_THT:TO-92L_Inline_Wide
- removed R20, R24: 22K, Resistor_SMD:R_0805_2012Metric_Pad1.20x1.40mm_HandSolder
- removed R21, R23, R25, R27: 3.3K, Resistor_SMD:R_0805_2012Metric_Pad1.20x1.40mm_HandSolder
- removed R22, R26: 100K, Resistor_SMD:R_0805_2012Metric_Pad1.20x1.40mm_HandSolder
- C3: footprint Capacitor_THT:CP_Radial_D5.0mm_P2.50mm -> Capacitor_THT:CP_Radial_D8.0mm_P3.50mm
- L1: footprint Inductor_THT:L_Radial_D7.2mm_P3.00mm_MuRATA_1700 -> Inductor_THT:L_Radial_D12.5mm_P7.00mm_Fastron_09HCP
- R12, R4, R8: footprint Resistor_SMD:R_0805_2012Metric_Pad1.20x1.40mm_HandSolder -> Resistor_SMD:R_1206_3216Metric_Pad1.30x1.75mm_HandSolder
- R16: value 22K -> 3.3K
- R17: value 3.3K -> 100K
- R18: value 100K -> 3.3K
- R19: value 3.3K -> 22K; footprint Resistor_SMD:R_0805_2012Metric_Pad1.20x1.40mm_HandSolder -> Resistor_SMD:R_1206_3216Metric_Pad1.30x1.75mm_HandSolder
- moved R41 67.8 mm to (121.5, 81.3), turned to 0 degrees
- moved NE1 64.0 mm to (120.5, 88.3), turned to 180 degrees
- moved R40 63.9 mm to (126.0, 79.3), turned to 0 degrees
- moved NE2 56.9 mm to (127.3, 77.3), turned to 135 degrees
- moved R34 56.6 mm to (142.0, 49.3), turned to 180 degrees
- moved R36 55.0 mm to (180.5, 49.3), turned to 180 degrees
- moved Q6 51.3 mm to (185.0, 96.1), turned to 180 degrees
- moved NE8 50.5 mm to (142.2, 52.2)
- moved R9 50.0 mm to (187.5, 87.3), turned to 270 degrees
- moved R39 49.1 mm to (143.5, 75.8), turned to 180 degrees
- moved R10 48.7 mm to (185.8, 91.8), turned to 180 degrees
- moved NE3 47.7 mm to (139.8, 71.6), turned to 90 degrees
- moved Q4 47.6 mm to (140.0, 92.3), turned to 180 degrees
- moved NE6 47.1 mm to (176.0, 44.2)
- moved R11 45.7 mm to (180.0, 91.8)
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Connections:
- J2 pad 12: idig5 -> Net-(J2-Pad12)
- J2 pad 14: idig6 -> Net-(J2-Pad14)
- NE1 pad 1: dig6 -> dig4
- NE10 pad 1: dig6 -> dig4
- NE2 pad 1: dig6 -> dig4
- NE3 pad 1: dig6 -> dig4
- NE4 pad 1: dig6 -> dig4
- NE5 pad 1: dig6 -> dig4
- NE6 pad 1: dig6 -> dig4
- NE7 pad 1: dig6 -> dig4
- NE8 pad 1: dig6 -> dig4
- NE9 pad 1: dig6 -> dig4
- Q8 pad 3: Net-(Q8-Pad3) -> dig4
- R13 pad 2: idig3 -> idig4
- R16 pad 1: dig3 -> Net-(Q9-Pad2)
- R16 pad 2: Net-(Q8-Pad3) -> idig3
- R17 pad 1: Net-(Q9-Pad2) -> 160V
- R17 pad 2: idig4 -> Net-(Q10-Pad2)
- R18 pad 1: 160V -> Net-(Q9-Pad1)
- R18 pad 2: Net-(Q10-Pad2) -> GNDREF
- R19 pad 1: Net-(Q9-Pad1) -> dig3
- R19 pad 2: GNDREF -> Net-(Q10-Pad3)
Routing:
- net GNDREF: track 557.8 -> 13.5 mm, vias 112 -> 39
- net dig6: track 195.7 -> 0.00 mm, vias 6 -> 0
- net dig4: track 18.1 -> 187.9 mm
- net 160V: track 244.9 -> 172.3 mm, vias 2 -> 0
- net /seg0: track 153.2 -> 101.0 mm, vias 8 -> 1
- net idig5: track 50.8 -> 0.00 mm, vias 1 -> 0
- net /seg6: track 141.8 -> 92.4 mm, vias 0 -> 1
- net /seg4: track 151.0 -> 104.0 mm
- net /seg3: track 149.2 -> 103.0 mm
- net /seg2: track 144.9 -> 103.7 mm, vias 1 -> 3
- net /seg8: track 127.4 -> 88.6 mm, vias 9 -> 2
- net /seg9: track 137.3 -> 102.6 mm, vias 6 -> 5
- net /seg5: track 129.7 -> 99.6 mm, vias 1 -> 0
- net dig3: track 16.1 -> 43.5 mm, vias 2 -> 1
- net /seg1: track 133.7 -> 106.4 mm, vias 7 -> 1
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- added copper zone on F.Cu, net GNDREF
