File: esp32/touch-panel2/touch-panel2.kicad_pcb (KiCad board)
At the start: 2 copper layers, 31.2 x 31.7 mm, 9 parts, among them J1 Conn_01x05, U1 AT42Q2120

Commit message: Fixed keywords for PCB
[git-p4: depot-paths = "//depot/nixiestat/": change = 358]
Other:
- board text added: "$Revision$"
- board text removed: "$Id$"
